Commit message: switched upper/lower on joints so upper is larger - moveit works now

File: inmoov_description/urdf/config.joints.urdf.xacro (robot description, xacro)
@@ -14,6 +14,6 @@
   <xacro:property name="r_middle_joint_upper"            value="${r*c['joints']['r_middle_joint']['maxGoal']}" />
   <xacro:property name="r_middle_joint_velocity"         value="${r*c['joints']['r_middle_joint']['maxSpeed']}" />
-  <xacro:property name="r_shoulder_lift_joint_lower"     value="${r*c['joints']['r_shoulder_lift_joint']['minGoal']}" />
-  <xacro:property name="r_shoulder_lift_joint_upper"     value="${r*c['joints']['r_shoulder_lift_joint']['maxGoal']}" />
+  <xacro:property name="r_shoulder_lift_joint_upper"     value="${r*c['joints']['r_shoulder_lift_joint']['minGoal']}" />
+  <xacro:property name="r_shoulder_lift_joint_lower"     value="${r*c['joints']['r_shoulder_lift_joint']['maxGoal']}" />
   <xacro:property name="r_shoulder_lift_joint_velocity"  value="${r*c['joints']['r_shoulder_lift_joint']['maxSpeed']}" />
   <xacro:property name="l_ring_joint_lower"              value="${r*c['joints']['l_ring_joint']['minGoal']}" />
@@ -26,9 +26,9 @@
   <xacro:property name="head_roll_joint_upper"           value="${r*c['joints']['head_roll_joint']['maxGoal']}" />
   <xacro:property name="head_roll_joint_velocity"        value="${r*c['joints']['head_roll_joint']['maxSpeed']}" />
-  <xacro:property name="waist_roll_joint_lower"          value="${r*c['joints']['waist_roll_joint']['minGoal']}" />
-  <xacro:property name="waist_roll_joint_upper"          value="${r*c['joints']['waist_roll_joint']['maxGoal']}" />
+  <xacro:property name="waist_roll_joint_upper"          value="${r*c['joints']['waist_roll_joint']['minGoal']}" />
+  <xacro:property name="waist_roll_joint_lower"          value="${r*c['joints']['waist_roll_joint']['maxGoal']}" />
   <xacro:property name="waist_roll_joint_velocity"       value="${r*c['joints']['waist_roll_joint']['maxSpeed']}" />
-  <xacro:property name="r_wrist_roll_joint_lower"        value="${r*c['joints']['r_wrist_roll_joint']['minGoal']}" />
-  <xacro:property name="r_wrist_roll_joint_upper"        value="${r*c['joints']['r_wrist_roll_joint']['maxGoal']}" />
+  <xacro:property name="r_wrist_roll_joint_upper"        value="${r*c['joints']['r_wrist_roll_joint']['minGoal']}" />
+  <xacro:property name="r_wrist_roll_joint_lower"        value="${r*c['joints']['r_wrist_roll_joint']['maxGoal']}" />
   <xacro:property name="r_wrist_roll_joint_velocity"     value="${r*c['joints']['r_wrist_roll_joint']['maxSpeed']}" />
   <xacro:property name="l_middle_joint_lower"            value="${r*c['joints']['l_middle_joint']['minGoal']}" />
@@ -38,15 +38,15 @@
   <xacro:property name="l_thumb_joint_upper"             value="${r*c['joints']['l_thumb_joint']['maxGoal']}" />
   <xacro:property name="l_thumb_joint_velocity"          value="${r*c['joints']['l_thumb_joint']['maxSpeed']}" />
-  <xacro:property name="l_elbow_flex_joint_lower"        value="${r*c['joints']['l_elbow_flex_joint']['minGoal']}" />
-  <xacro:property name="l_elbow_flex_joint_upper"        value="${r*c['joints']['l_elbow_flex_joint']['maxGoal']}" />
+  <xacro:property name="l_elbow_flex_joint_upper"        value="${r*c['joints']['l_elbow_flex_joint']['minGoal']}" />
+  <xacro:property name="l_elbow_flex_joint_lower"        value="${r*c['joints']['l_elbow_flex_joint']['maxGoal']}" />
   <xacro:property name="l_elbow_flex_joint_velocity"     value="${r*c['joints']['l_elbow_flex_joint']['maxSpeed']}" />
   <xacro:property name="jaw_joint_lower"                 value="${r*c['joints']['jaw_joint']['minGoal']}" />
   <xacro:property name="jaw_joint_upper"                 value="${r*c['joints']['jaw_joint']['maxGoal']}" />
   <xacro:property name="jaw_joint_velocity"              value="${r*c['joints']['jaw_joint']['maxSpeed']}" />
-  <xacro:property name="l_wrist_roll_joint_lower"        value="${r*c['joints']['l_wrist_roll_joint']['minGoal']}" />
-  <xacro:property name="l_wrist_roll_joint_upper"        value="${r*c['joints']['l_wrist_roll_joint']['maxGoal']}" />
+  <xacro:property name="l_wrist_roll_joint_upper"        value="${r*c['joints']['l_wrist_roll_joint']['minGoal']}" />
+  <xacro:property name="l_wrist_roll_joint_lower"        value="${r*c['joints']['l_wrist_roll_joint']['maxGoal']}" />
   <xacro:property name="l_wrist_roll_joint_velocity"     value="${r*c['joints']['l_wrist_roll_joint']['maxSpeed']}" />
-  <xacro:property name="r_elbow_flex_joint_lower"        value="${r*c['joints']['r_elbow_flex_joint']['minGoal']}" />
-  <xacro:property name="r_elbow_flex_joint_upper"        value="${r*c['joints']['r_elbow_flex_joint']['maxGoal']}" />
+  <xacro:property name="r_elbow_flex_joint_upper"        value="${r*c['joints']['r_elbow_flex_joint']['minGoal']}" />
+  <xacro:property name="r_elbow_flex_joint_lower"        value="${r*c['joints']['r_elbow_flex_joint']['maxGoal']}" />
   <xacro:property name="r_elbow_flex_joint_velocity"     value="${r*c['joints']['r_elbow_flex_joint']['maxSpeed']}" />
   <xacro:property name="eyes_pan_joint_lower"            value="${r*c['joints']['eyes_pan_joint']['minGoal']}" />
@@ -56,9 +56,9 @@
   <xacro:property name="r_ring_joint_upper"              value="${r*c['joints']['r_ring_joint']['maxGoal']}" />
   <xacro:property name="r_ring_joint_velocity"           value="${r*c['joints']['r_ring_joint']['maxSpeed']}" />
-  <xacro:property name="l_shoulder_lift_joint_lower"     value="${r*c['joints']['l_shoulder_lift_joint']['minGoal']}" />
-  <xacro:property name="l_shoulder_lift_joint_upper"     value="${r*c['joints']['l_shoulder_lift_joint']['maxGoal']}" />
+  <xacro:property name="l_shoulder_lift_joint_upper"     value="${r*c['joints']['l_shoulder_lift_joint']['minGoal']}" />
+  <xacro:property name="l_shoulder_lift_joint_lower"     value="${r*c['joints']['l_shoulder_lift_joint']['maxGoal']}" />
   <xacro:property name="l_shoulder_lift_joint_velocity"  value="${r*c['joints']['l_shoulder_lift_joint']['maxSpeed']}" />
-  <xacro:property name="eyes_tilt_joint_lower"           value="${r*c['joints']['eyes_tilt_joint']['minGoal']}" />
-  <xacro:property name="eyes_tilt_joint_upper"           value="${r*c['joints']['eyes_tilt_joint']['maxGoal']}" />
+  <xacro:property name="eyes_tilt_joint_upper"           value="${r*c['joints']['eyes_tilt_joint']['minGoal']}" />
+  <xacro:property name="eyes_tilt_joint_lower"           value="${r*c['joints']['eyes_tilt_joint']['maxGoal']}" />
   <xacro:property name="eyes_tilt_joint_velocity"        value="${r*c['joints']['eyes_tilt_joint']['maxSpeed']}" />
   <xacro:property name="r_index_joint_lower"             value="${r*c['joints']['r_index_joint']['minGoal']}" />
@@ -83,6 +83,6 @@
   <xacro:property name="r_thumb_joint_upper"             value="${r*c['joints']['r_thumb_joint']['maxGoal']}" />
   <xacro:property name="r_thumb_joint_velocity"          value="${r*c['joints']['r_thumb_joint']['maxSpeed']}" />
-  <xacro:property name="r_upper_arm_roll_joint_lower"    value="${r*c['joints']['r_upper_arm_roll_joint']['minGoal']}" />
-  <xacro:property name="r_upper_arm_roll_joint_upper"    value="${r*c['joints']['r_upper_arm_roll_joint']['maxGoal']}" />
+  <xacro:property name="r_upper_arm_roll_joint_upper"    value="${r*c['joints']['r_upper_arm_roll_joint']['minGoal']}" />
+  <xacro:property name="r_upper_arm_roll_joint_lower"    value="${r*c['joints']['r_upper_arm_roll_joint']['maxGoal']}" />
   <xacro:property name="r_upper_arm_roll_joint_velocity" value="${r*c['joints']['r_upper_arm_roll_joint']['maxSpeed']}" />
   <xacro:property name="l_upper_arm_roll_joint_lower"    value="${r*c['joints']['l_upper_arm_roll_joint']['minGoal']}" />
@@ -92,6 +92,6 @@
   <xacro:property name="head_tilt_joint_upper"           value="${r*c['joints']['head_tilt_joint']['maxGoal']}" />
   <xacro:property name="head_tilt_joint_velocity"        value="${r*c['joints']['head_tilt_joint']['maxSpeed']}" />
-  <xacro:property name="r_shoulder_out_joint_lower"      value="${r*c['joints']['r_shoulder_out_joint']['minGoal']}" />
-  <xacro:property name="r_shoulder_out_joint_upper"      value="${r*c['joints']['r_shoulder_out_joint']['maxGoal']}" />
+  <xacro:property name="r_shoulder_out_joint_upper"      value="${r*c['joints']['r_shoulder_out_joint']['minGoal']}" />
+  <xacro:property name="r_shoulder_out_joint_lower"      value="${r*c['joints']['r_shoulder_out_joint']['maxGoal']}" />
   <xacro:property name="r_shoulder_out_joint_velocity"   value="${r*c['joints']['r_shoulder_out_joint']['maxSpeed']}" />
 </robot>
